File: Hardware/ST-Link_v2-1/ST-Link_v2-1.sch (KiCad schematic (older format))
At the start: 4 parts

Commit message: 16-11-2021
Parts:
- removed J?: Conn_01x04, HKUST_RT_Conn:Molex_SL_171971-0004_1x04_P2.54mm_Vertical, symbol HKUST_RT_CONN:Conn_01x04
- added C? (x2): 1uF, HKUST_RT_RCL:C_0805_2012Metric_Pad1.18x1.45mm_HandSolder, symbol HKUST_RT_RCL:C_Small
- added C? (x7): C_Small, HKUST_RT_RCL:C_0805_2012Metric_Pad1.18x1.45mm_HandSolder, symbol HKUST_RT_RCL:C_Small
- added D? (x5): LED_Small, HKUST_RT_BJT:LED_0805_2012Metric_Pad1.15x1.40mm_HandSolder, symbol HKUST_RT_BJT:LED_Small
- added D? (x2): 1N4001, Diode_THT:D_DO-41_SOD81_P10.16mm_Horizontal, symbol HKUST_RT_BJT:1N4001
- added J?: Conn_01x06, symbol HKUST_RT_CONN:Conn_01x06
- added JP? (x2): SolderJumper_2_Open, symbol HKUST_RT_CONN:SolderJumper_2_Open
- added R? (x14): R_Small_US, HKUST_RT_RCL:R_0805_2012Metric_Pad1.20x1.40mm_HandSolder, symbol HKUST_RT_RCL:R_Small_US
- added Y?: Crystal_Small, symbol HKUST_RT_RCL:Crystal_Small
Connections:
- net labels added: +3.3V, +5V, GND
- wire segments 0 -> 25
- no-connect marks 0 -> 12
Other:
- moved on the sheet: U?

Commit message: 18-11-2021
Parts:
- added R? (x2): 10k, HKUST_RT_RCL:R_0805_2012Metric_Pad1.20x1.40mm_HandSolder, symbol HKUST_RT_RCL:R_Small_US
- C? (x2): value C_Small -> 22pF
- C? (x5): value C_Small -> 100nF
- D?: value LED_Small -> 3.3V
- D?: value LED_Small -> TX
- D?: value LED_Small -> RX
- R? (x5): value R_Small_US -> 1.5k
- R?: value R_Small_US -> 10k
- R? (x2): value R_Small_US -> 100R
- R?: value R_Small_US -> 100k
- R? (x3): value R_Small_US -> 4.7k
- R? (x2): value R_Small_US -> 22R
- Y?: value Crystal_Small -> 8MHz
Connections:
- net labels added: D+, D-, LED_STLINK, NRST, RXD, ST_SWCLK, ST_SWDIO, SWCLK, SWDIO, SWDIO_IN, TXD, USB_RENUMn
- wire segments 25 -> 76
- no-connect marks 12 -> 29
Other:
- moved on the sheet: C?, D?, J?, R?, U?

Commit message: 20-11-2021
Parts:
- removed D?: 1N4001, Diode_THT:D_DO-41_SOD81_P10.16mm_Horizontal, symbol HKUST_RT_BJT:1N4001
- removed JP? (x2): SolderJumper_2_Open, symbol HKUST_RT_CONN:SolderJumper_2_Open
- added R13: 100R, HKUST_RT_RCL:R_0402_1005Metric, symbol HKUST_RT_RCL:R_Small_US
- added R16: 1.5k, HKUST_RT_RCL:R_0402_1005Metric, symbol HKUST_RT_RCL:R_Small_US
- added R19, R20: 0R, HKUST_RT_RCL:R_0402_1005Metric, symbol HKUST_RT_RCL:R_Small_US
- C1, C2, C3, C4, C5, C6, C7, C8, C9: renamed from C?; footprint HKUST_RT_RCL:C_0805_2012Metric_Pad1.18x1.45mm_HandSolder -> HKUST_RT_RCL:C_0402_1005Metric
- D1, D2, D3, D4, D5: renamed from D?; footprint HKUST_RT_BJT:LED_0805_2012Metric_Pad1.15x1.40mm_HandSolder -> HKUST_RT_BJT:LED_0402_1005Metric
- D6: renamed from D?; footprint Diode_THT:D_DO-41_SOD81_P10.16mm_Horizontal -> HKUST_RT_BJT:D_SMA
- J1: renamed from J?; footprint (none) -> HKUST_RT_CONN:JST_GH_SM06B-GHS-TB_1x06-1MP_P1.25mm_Horizontal
- P1: renamed from P?; footprint (none) -> HKUST_RT_CONN:USB_C_Plug_Molex_105444
- R1, R10, R11, R12, R14, R15, R17, R18, R2, R3, R4, R5, R6, R7, R8, R9: renamed from R?; footprint HKUST_RT_RCL:R_0805_2012Metric_Pad1.20x1.40mm_HandSolder -> HKUST_RT_RCL:R_0402_1005Metric
- U1: renamed from U?; footprint Package_QFP:LQFP-48_7x7mm_P0.5mm -> HKUST_RT_IC:LQFP-48_7x7mm_P0.5mm
- Y1: renamed from Y?; footprint (none) -> HKUST_RT_RCL:Crystal_SMD_3225-4Pin_3.2x2.5mm
- gave numbers to parts that had none: 1
Connections:
- net labels removed: USB_RENUMn
- wire segments 76 -> 77

Commit message: 21-11-2021
Parts:
- removed P1: USB_C_Plug, HKUST_RT_CONN:USB_C_Plug_Molex_105444, symbol HKUST_RT_CONN:USB_C_Plug
- added J2: USB_C_Male, HKUST_RT_CONN:USB_C_MALE, symbol HKUST_RT_CONN:USB_C_Male
- D6: footprint HKUST_RT_BJT:D_SMA -> HKUST_RT_BJT:D_0402_1005Metric
- U2: footprint Package_TO_SOT_SMD:SOT-23-5 -> HKUST_RT_IC:SOT-23-5
Connections:
- wire segments 77 -> 78
Other:
- moved on the sheet: R16, R17, R18
Changed lines of the file:
@@
 F 0 "U2" H 5950 5217 50  0000 C CNN
 F 1 "LP5907MFX-3.3" H 5950 5126 50  0000 C CNN
-F 2 "Package_TO_SOT_SMD:SOT-23-5" H 5950 5200 50  0001 C CNN
+F 2 "HKUST_RT_IC:SOT-23-5" H 5950 5200 50  0001 C CNN
 F 3 "" H 5950 5350 50  0001 C CNN
 	1    5950 4850
@@
 Wire Wire Line
 	2050 5150 1750 5150
-NoConn ~ 6450 2950
-NoConn ~ 6450 3050
-NoConn ~ 6450 2650
-NoConn ~ 6450 2750
-NoConn ~ 6450 2350
-NoConn ~ 6450 2450
-NoConn ~ 6450 2050
-NoConn ~ 6450 2150
-NoConn ~ 6450 3250
-NoConn ~ 6450 3350
-NoConn ~ 6450 1250
-NoConn ~ 6450 1350
 $Comp
 L power:GND #PWR022
 U 1 1 619A3AC9
-P 5550 3650
-F 0 "#PWR022" H 5550 3400 50  0001 C CNN
-F 1 "GND" H 5555 3477 50  0000 C CNN
-F 2 "" H 5550 3650 50  0001 C CNN
-F 3 "" H 5550 3650 50  0001 C CNN
-	1    5550 3650
-	1    0    0    -1
-$EndComp
-Wire Wire Line
-	5550 3650 5850 3650
+P 5650 2200
+F 0 "#PWR022" H 5650 1950 50  0001 C CNN
+F 1 "GND" H 5655 2027 50  0000 C CNN
+F 2 "" H 5650 2200 50  0001 C CNN
+F 3 "" H 5650 2200 50  0001 C CNN
+	1    5650 2200
+	0    1    1    0
+$EndComp
 $Comp
 L power:+5V #PWR028
 U 1 1 619A512D
-P 6750 1050
-F 0 "#PWR028" H 6750 900 50  0001 C CNN
-F 1 "+5V" V 6765 1178 50  0000 L CNN
-F 2 "" H 6750 1050 50  0001 C CNN
-F 3 "" H 6750 1050 50  0001 C CNN
-	1    6750 1050
-	0    1    1    0
+P 5700 1100
+F 0 "#PWR028" H 5700 950 50  0001 C CNN
+F 1 "+5V" V 5800 1100 50  0000 L CNN
+F 2 "" H 5700 1100 50  0001 C CNN
+F 3 "" H 5700 1100 50  0001 C CNN
+	1    5700 1100
+	0    -1   -1   0
 $EndComp
 $Comp
 L HKUST_RT_RCL:R_Small_US R17
 U 1 1 619A5D6F
-P 6750 1550
-F 0 "R17" V 6850 1550 50  0000 C CNN
-F 1 "22R" V 6800 1700 50  0000 C CNN
-F 2 "HKUST_RT_RCL:R_0402_1005Metric" H 6818 1459 50  0001 L CNN
-F 3 "" H 6750 1550 50  0001 C CNN
-	1    6750 1550
-	0    -1   -1   0
+P 5400 1600
+F 0 "R17" V 5500 1600 50  0000 C CNN
+F 1 "22R" V 5450 1750 50  0000 C CNN
+F 2 "HKUST_RT_RCL:R_0402_1005Metric" H 5468 1509 50  0001 L CNN
+F 3 "" H 5400 1600 50  0001 C CNN
+	1    5400 1600
+	0    1    1    0
 $EndComp
 $Comp
 L HKUST_RT_RCL:R_Small_US R18
 U 1 1 619A63BA
-P 6750 1750
-F 0 "R18" V 6850 1750 50  0000 C CNN
-F 1 "22R" V 6800 1900 50  0000 C CNN
-F 2 "HKUST_RT_RCL:R_0402_1005Metric" H 6818 1659 50  0001 L CNN
-F 3 "" H 6750 1750 50  0001 C CNN
-	1    6750 1750
-	0    -1   -1   0
-$EndComp
-Connection ~ 5550 3650
-$Comp
-L HKUST_RT_CONN:USB_C_Plug P1
-U 1 1 619061E1
-P 5850 2050
-F 0 "P1" H 5957 3317 50  0000 C CNN
-F 1 "USB_C_Plug" H 5957 3226 50  0000 C CNN
-F 2 "HKUST_RT_CONN:USB_C_Plug_Molex_105444" H 6000 2050 50  0001 C CNN
-F 3 "https://www.usb.org/sites/default/files/documents/usb_type-c.zip" H 6000 2050 50  0001 C CNN
-	1    5850 2050
-	1    0    0    -1
-$EndComp
-Wire Wire Line
-	6450 1050 6750 1050
+P 5400 1500
+F 0 "R18" V 5350 1350 50  0000 C CNN
+F 1 "22R" V 5450 1650 50  0000 C CNN
+F 2 "HKUST_RT_RCL:R_0402_1005Metric" H 5468 1409 50  0001 L CNN
+F 3 "" H 5400 1500 50  0001 C CNN
+	1    5400 1500
+	0    1    1    0
+$EndComp
 Wire Wire Line
 	3000 7050 3000 6650
@@
 	3000 6650 3650 6650
 Wire Wire Line
-	6450 1550 6650 1550
-Wire Wire Line
-	6450 1750 6600 1750
+	5700 1600 5500 1600
+Wire Wire Line
+	5700 1500 5550 1500
 Text Label 2550 7050 0    50   ~ 0
 LED_STLINK
@@
 	4600 500  4600 7750
 Wire Wire Line
-	7350 1550 6850 1550
-Wire Wire Line
-	7350 1750 6850 1750
-Text Label 7100 1550 0    50   ~ 0
+	4800 1600 5300 1600
+Wire Wire Line
+	4800 1500 5300 1500
+Text Label 5050 1600 2    50   ~ 0
 D-
-Text Label 7100 1750 0    50   ~ 0
+Text Label 5050 1500 2    50   ~ 0
 D+
-Connection ~ 6600 1750
-Wire Wire Line
-	6600 1750 6650 1750
+Connection ~ 5550 1500
+Wire Wire Line
+	5550 1500 5500 1500
 $Comp
 L HKUST_RT_RCL:R_Small_US R16
 U 1 1 6196ADF3
-P 6600 1850
-F 0 "R16" H 6700 1850 50  0000 C CNN
-F 1 "1.5k" H 6700 1750 50  0000 C CNN
-F 2 "HKUST_RT_RCL:R_0402_1005Metric" H 6668 1759 50  0001 L CNN
-F 3 "" H 6600 1850 50  0001 C CNN
-	1    6600 1850
-	1    0    0    -1
+P 5550 1400
+F 0 "R16" H 5450 1450 50  0000 C CNN
+F 1 "1.5k" H 5700 1350 50  0000 C CNN
+F 2 "HKUST_RT_RCL:R_0402_1005Metric" H 5618 1309 50  0001 L CNN
+F 3 "" H 5550 1400 50  0001 C CNN
+	1    5550 1400
+	-1   0    0    1
 $EndComp
 $Comp
 L power:+3.3V #PWR027
 U 1 1 6196BFC6
-P 6600 1950
-F 0 "#PWR027" H 6600 1800 50  0001 C CNN
-F 1 "+3.3V" H 6615 2123 50  0000 C CNN
-F 2 "" H 6600 1950 50  0001 C CNN
-F 3 "" H 6600 1950 50  0001 C CNN
-	1    6600 1950
-	-1   0    0    1
+P 5550 1300
+F 0 "#PWR027" H 5550 1150 50  0001 C CNN
+F 1 "+3.3V" H 5350 1400 50  0000 C CNN
+F 2 "" H 5550 1300 50  0001 C CNN
+F 3 "" H 5550 1300 50  0001 C CNN
+	1    5550 1300
+	1    0    0    -1
 $EndComp
 $Comp
@@
 F 0 "D6" H 5750 6950 50  0000 C CNN
 F 1 "1N4001" H 6000 6950 50  0000 C CNN
-F 2 "HKUST_RT_BJT:D_SMA" H 6000 6925 50  0001 C CNN
+F 2 "HKUST_RT_BJT:D_0402_1005Metric" H 6000 6925 50  0001 C CNN
 F 3 "http://www.vishay.com/docs/88503/1n4001.pdf" H 6000 7100 50  0001 C CNN
 	1    6000 7100
@@
 	1    0    0    -1
 $EndComp
+$Comp
+L HKUST_RT_CONN:USB_C_Male J2
+U 1 1 619AAADA
+P 6500 1600
+F 0 "J2" H 6500 2367 50  0000 C CNN
+F 1 "USB_C_Male" H 6500 2276 50  0000 C CNN
+F 2 "HKUST_RT_CONN:USB_C_MALE" H 6500 1600 50  0001 L BNN
+F 3 "" H 6500 1600 50  0001 L BNN
+F 4 "Hirose" H 6500 1600 50  0001 L BNN "MANUFACTURER"
+F 5 "5" H 6500 1600 50  0001 L BNN "PARTREV"
+F 6 "Manufacturer Recommendations" H 6500 1600 50  0001 L BNN "STANDARD"
+F 7 "2.6 mm" H 6500 1600 50  0001 L BNN "MAXIMUM_PACKAGE_HEIGHT"
+	1    6500 1600
+	1    0    0    -1
+$EndComp
+NoConn ~ 5700 1200
+NoConn ~ 5700 1300
+NoConn ~ 5700 1400
+NoConn ~ 5700 1700
+NoConn ~ 5700 1800
+NoConn ~ 5700 1900
+Wire Wire Line
+	5700 2000 5700 2200
+Wire Wire Line
+	5650 2200 5700 2200
+Connection ~ 5700 2200
+Wire Wire Line
+	7300 2000 7300 2200
+$Comp
+L power:GND #PWR0102
+U 1 1 619EB02D
+P 7300 2200
+F 0 "#PWR0102" H 7300 1950 50  0001 C CNN
+F 1 "GND" H 7305 2027 50  0000 C CNN
+F 2 "" H 7300 2200 50  0001 C CNN
+F 3 "" H 7300 2200 50  0001 C CNN
+	1    7300 2200
+	0    -1   -1   0
+$EndComp
+Connection ~ 7300 2200
+NoConn ~ 7300 1700
+NoConn ~ 7300 1800
+NoConn ~ 7300 1900
+NoConn ~ 7300 1400
+NoConn ~ 7300 1300
+NoConn ~ 7300 1200
+$Comp
+L power:+5V #PWR0103
+U 1 1 619F8999
+P 7300 1100
+F 0 "#PWR0103" H 7300 950 50  0001 C CNN
+F 1 "+5V" V 7300 1250 50  0000 L CNN
+F 2 "" H 7300 1100 50  0001 C CNN
+F 3 "" H 7300 1100 50  0001 C CNN
+	1    7300 1100
+	0    1    1    0
+$EndComp
 $EndSCHEMATC

Commit message: v2 2/12/2021
Parts:
- added R21: 5.1k, HKUST_RT_RCL:R_0805_2012Metric_Pad1.20x1.40mm_HandSolder, symbol HKUST_RT_RCL:R_Small_US
- C1, C2, C3, C4, C5, C6, C7, C8, C9: footprint HKUST_RT_RCL:C_0402_1005Metric -> HKUST_RT_RCL:C_0805_2012Metric_Pad1.18x1.45mm_HandSolder
- D1, D2, D3, D4, D5: footprint HKUST_RT_BJT:LED_0402_1005Metric -> HKUST_RT_BJT:LED_0805_2012Metric_Pad1.15x1.40mm_HandSolder
- D6: footprint HKUST_RT_BJT:D_0402_1005Metric -> HKUST_RT_BJT:D_SOD-123
- R1, R10, R11, R12, R13, R14, R15, R16, R17, R18, R2, R3, R4, R5, R6, R7, R8, R9: footprint HKUST_RT_RCL:R_0402_1005Metric -> HKUST_RT_RCL:R_0805_2012Metric_Pad1.20x1.40mm_HandSolder
Connections:
- wire segments 78 -> 82
- no-connect marks 29 -> 28
Other:
- moved on the sheet: D6

Commit message: find bug in sch
Parts:
- removed J2: USB_C_Male, HKUST_RT_CONN:USB_C_MALE, symbol HKUST_RT_CONN:USB_C_Male
- removed Y1: 8MHz, HKUST_RT_RCL:Crystal_SMD_3225-4Pin_3.2x2.5mm, symbol HKUST_RT_RCL:Crystal_Small
- added J2: USB_C_Receptacle, HKUST_RT_CONN:USB_C_MALE, symbol HKUST_RT_CONN:USB_C_Receptacle
- added R22: 5.1k, HKUST_RT_RCL:R_0805_2012Metric, symbol HKUST_RT_RCL:R_Small_US
- added Y1: 8Mhz, HKUST_RT_RCL:Crystal_SMD_3225-4Pin_3.2x2.5mm, symbol HKUST_RT_RCL:Crystal_GND24_Small
- C1, C2, C3, C4, C5, C6, C7, C8, C9: footprint HKUST_RT_RCL:C_0805_2012Metric_Pad1.18x1.45mm_HandSolder -> HKUST_RT_RCL:C_0805_2012Metric
- D1, D2, D3, D4, D5: footprint HKUST_RT_BJT:LED_0805_2012Metric_Pad1.15x1.40mm_HandSolder -> HKUST_RT_BJT:LED_0805_2012Metric
- R1, R10, R11, R12, R13, R14, R15, R16, R17, R18, R2, R21, R3, R4, R5, R6, R8, R9: footprint HKUST_RT_RCL:R_0805_2012Metric_Pad1.20x1.40mm_HandSolder -> HKUST_RT_RCL:R_0805_2012Metric
- R19, R20: footprint HKUST_RT_RCL:R_0402_1005Metric -> HKUST_RT_RCL:R_0805_2012Metric
- R7: value 100R -> 10k; footprint HKUST_RT_RCL:R_0805_2012Metric_Pad1.20x1.40mm_HandSolder -> HKUST_RT_RCL:R_0805_2012Metric
Connections:
- wire segments 82 -> 77
- no-connect marks 28 -> 27
Other:
- moved on the sheet: D6, R16, R17, R18, R21

Commit message: 5/12/2021
Parts:
- removed D6: 1N4001, HKUST_RT_BJT:D_SOD-123, symbol HKUST_RT_BJT:1N4001
- removed R13: 100R, HKUST_RT_RCL:R_0805_2012Metric, symbol HKUST_RT_RCL:R_Small_US
- R14, R15: value 4.7k -> 10k
Connections:
- net labels added: JTCK, JTMS
- net labels removed: SWCLK, SWDIO, SWDIO_IN
- wire segments 77 -> 72
- no-connect marks 27 -> 28
Changed lines of the file:
@@
 $EndDescr
-$Comp
-L HKUST_RT_IC:STM32F103CBTx U1
-U 1 1 618FB8D3
-P 2700 3050
-F 0 "U1" H 2950 1500 50  0000 C CNN
-F 1 "STM32F103CBTx" H 3300 1500 50  0000 C CNN
-F 2 "HKUST_RT_IC:LQFP-48_7x7mm_P0.5mm" H 2100 1650 50  0001 R CNN
-F 3 "http://www.st.com/st-web-ui/static/active/en/resource/technical/document/datasheet/CD00161566.pdf" H 2700 3050 50  0001 C CNN
-	1    2700 3050
-	1    0    0    -1
-$EndComp
 $Comp
 L HKUST_RT_IC:LP5907MFX-3.3 U2
@@
 P 4050 2950
 F 0 "R15" H 3982 2904 50  0000 R CNN
-F 1 "4.7k" H 3982 2995 50  0000 R CNN
+F 1 "10k" H 3982 2995 50  0000 R CNN
 F 2 "HKUST_RT_RCL:R_0805_2012Metric" H 4118 2859 50  0001 L CNN
 F 3 "" H 4050 2950 50  0001 C CNN
@@
 	2000 1400 2000 1750
 Connection ~ 950  1400
-Wire Wire Line
-	2800 4550 2700 4550
-Connection ~ 2500 4550
-Connection ~ 2600 4550
-Wire Wire Line
-	2600 4550 2500 4550
-Connection ~ 2700 4550
-Wire Wire Line
-	2700 4550 2600 4550
-Wire Wire Line
-	2900 1550 2800 1550
-Connection ~ 2600 1550
-Wire Wire Line
-	2600 1550 2500 1550
-Connection ~ 2700 1550
-Wire Wire Line
-	2700 1550 2600 1550
-Connection ~ 2800 1550
-Wire Wire Line
-	2800 1550 2700 1550
 $Comp
 L power:+3.3V #PWR014
@@
 	1    0    0    -1
 $EndComp
-Connection ~ 2500 1550
 Wire Wire Line
 	3400 6800 3450 6800
@@
 P 4050 2750
 F 0 "R14" H 3982 2704 50  0000 R CNN
-F 1 "4.7k" H 3982 2795 50  0000 R CNN
+F 1 "10k" H 3982 2795 50  0000 R CNN
 F 2 "HKUST_RT_RCL:R_0805_2012Metric" H 4118 2659 50  0001 L CNN
 F 3 "" H 4050 2750 50  0001 C CNN
@@
 	3800 3150 3300 3150
 NoConn ~ 3300 3250
-NoConn ~ 3300 3450
-NoConn ~ 3300 3550
 NoConn ~ 2000 2950
-NoConn ~ 2000 3850
 NoConn ~ 2000 3950
 NoConn ~ 3300 3650
 NoConn ~ 2000 4350
-NoConn ~ 3300 3850
 NoConn ~ 2000 3250
 NoConn ~ 2000 3350
@@
 	0    1    1    0
 $EndComp
-$Comp
-L HKUST_RT_RCL:R_Small_US R10
-U 1 1 619A3D8D
-P 1900 2550
-F 0 "R10" V 2000 2550 50  0000 C CNN
-F 1 "10k" V 1950 2400 50  0000 C CNN
-F 2 "HKUST_RT_RCL:R_0805_2012Metric" H 1968 2459 50  0001 L CNN
-F 3 "" H 1900 2550 50  0001 C CNN
-	1    1900 2550
-	0    1    1    0
-$EndComp
-$Comp
-L power:GND #PWR012
-U 1 1 619A40C0
-P 1750 2500
-F 0 "#PWR012" H 1750 2250 50  0001 C CNN
-F 1 "GND" V 1755 2372 50  0000 R CNN
-F 2 "" H 1750 2500 50  0001 C CNN
-F 3 "" H 1750 2500 50  0001 C CNN
-	1    1750 2500
-	0    1    1    0
-$EndComp
-Wire Wire Line
-	1800 2500 1800 2450
-Wire Wire Line
-	1800 2550 1800 2500
-Wire Wire Line
-	1800 2500 1750 2500
-Connection ~ 1800 2500
 Wire Wire Line
 	1700 2850 2000 2850
@@
 NRST
 Text Label 5900 6900 0    50   ~ 0
-SWDIO
+JTMS
 Text Label 5900 7000 0    50   ~ 0
-SWCLK
+JTCK
 Wire Wire Line
 	6200 7000 5750 7000
@@
 	6300 5700 5850 5700
 Text Label 5350 5700 0    50   ~ 0
-SWCLK
+JTCK
 Text Label 5850 5700 0    50   ~ 0
 ST_SWCLK
 Text Label 5350 6000 0    50   ~ 0
-SWDIO
+JTMS
 Text Label 5850 6000 0    50   ~ 0
 ST_SWDIO
@@
 RXD
 Text Label 3500 3350 0    50   ~ 0
-SWCLK
-Text Label 1650 4250 0    50   ~ 0
-SWDIO
-Text Label 1600 4050 0    50   ~ 0
-SWDIO_IN
+JTCK
+Text Label 1600 4250 0    50   ~ 0
+JTMS
 Wire Wire Line
 	1600 4050 2000 4050
@@
 	1400 4250 2000 4250
 Text Label 1600 4150 0    50   ~ 0
-SWCLK
+JTCK
 $Comp
 L HKUST_RT_RCL:R_Small_US R2
@@
 Text Label 6700 1950 2    50   ~ 0
 D+
-$Comp
-L HKUST_RT_RCL:R_Small_US R13
-U 1 1 6196FBB1
-P 3600 4350
-F 0 "R13" V 3500 4300 50  0000 R CNN
-F 1 "100R" V 3500 4550 50  0000 R CNN
-F 2 "HKUST_RT_RCL:R_0805_2012Metric" H 3668 4259 50  0001 L CNN
-F 3 "" H 3600 4350 50  0001 C CNN
-	1    3600 4350
-	0    -1   -1   0
-$EndComp
-Wire Wire Line
-	3300 4350 3500 4350
 Wire Wire Line
 	6250 4750 6350 4750
@@
 L power:+5V #PWR0103
 U 1 1 619F8999
-P 6550 1150
-F 0 "#PWR0103" H 6550 1000 50  0001 C CNN
-F 1 "+5V" V 6550 1300 50  0000 L CNN
-F 2 "" H 6550 1150 50  0001 C CNN
-F 3 "" H 6550 1150 50  0001 C CNN
-	1    6550 1150
+P 6250 1150
+F 0 "#PWR0103" H 6250 1000 50  0001 C CNN
+F 1 "+5V" V 6250 1300 50  0000 L CNN
+F 2 "" H 6250 1150 50  0001 C CNN
+F 3 "" H 6250 1150 50  0001 C CNN
+	1    6250 1150
 	0    1    1    0
 $EndComp
@@
 	0    -1   -1   0
 $EndComp
-Wire Wire Line
-	6250 800  6250 1150
 $Comp
 L power:+5V #PWR021
@@
 	1    5250 4750
 	0    -1   -1   0
-$EndComp
-$Comp
-L power:PWR_FLAG #FLG0102
-U 1 1 61ABB2EF
-P 6250 800
-F 0 "#FLG0102" H 6250 875 50  0001 C CNN
-F 1 "PWR_FLAG" H 6250 973 50  0000 C CNN
-F 2 "" H 6250 800 50  0001 C CNN
-F 3 "~" H 6250 800 50  0001 C CNN
-	1    6250 800
-	1    0    0    -1
-$EndComp
-$Comp
-L HKUST_RT_BJT:1N4001 D6
-U 1 1 6199A377
-P 6400 1150
-F 0 "D6" H 6150 1000 50  0000 C CNN
-F 1 "1N4001" H 6400 1000 50  0000 C CNN
-F 2 "HKUST_RT_BJT:D_SOD-123" H 6400 975 50  0001 C CNN
-F 3 "http://www.vishay.com/docs/88503/1n4001.pdf" H 6400 1150 50  0001 C CNN
-	1    6400 1150
-	-1   0    0    1
 $EndComp
 Wire Wire Line
@@
 $EndComp
 Connection ~ 6250 1650
-Connection ~ 6250 1150
 Connection ~ 6250 1950
 NoConn ~ 6250 3150
-$Comp
-L power:+3.3V #PWR0106
-U 1 1 61B1CFDA
-P 3700 4350
-F 0 "#PWR0106" H 3700 4200 50  0001 C CNN
-F 1 "+3.3V" V 3700 4600 50  0000 C CNN
-F 2 "" H 3700 4350 50  0001 C CNN
-F 3 "" H 3700 4350 50  0001 C CNN
-	1    3700 4350
-	0    1    1    0
-$EndComp
+Wire Wire Line
+	2900 1550 2800 1550
+Connection ~ 2800 1550
+Wire Wire Line
+	2800 4550 2700 4550
+Connection ~ 2700 4550
+Wire Wire Line
+	2800 1550 2700 1550
+Connection ~ 2700 1550
+Wire Wire Line
+	2700 4550 2600 4550
+Wire Wire Line
+	2600 4550 2500 4550
+Connection ~ 2600 4550
+Wire Wire Line
+	2700 1550 2600 1550
+Wire Wire Line
+	2600 1550 2500 1550
+Connection ~ 2600 1550
+Connection ~ 2500 4550
+Connection ~ 2500 1550
+$Comp
+L HKUST_RT_IC:STM32F103CBTx U1
+U 1 1 618FB8D3
+P 2700 3050
+F 0 "U1" H 2950 1500 50  0000 C CNN
+F 1 "STM32F103CBTx" H 3300 1500 50  0000 C CNN
+F 2 "HKUST_RT_IC:LQFP-48_7x7mm_P0.5mm" H 2100 1650 50  0001 R CNN
+F 3 "http://www.st.com/st-web-ui/static/active/en/resource/technical/document/datasheet/CD00161566.pdf" H 2700 3050 50  0001 C CNN
+	1    2700 3050
+	1    0    0    -1
+$EndComp
+$Comp
+L power:GND #PWR0107
+U 1 1 61ACB3E8
+P 1800 2450
+F 0 "#PWR0107" H 1800 2200 50  0001 C CNN
+F 1 "GND" V 1805 2322 50  0000 R CNN
+F 2 "" H 1800 2450 50  0001 C CNN
+F 3 "" H 1800 2450 50  0001 C CNN
+	1    1800 2450
+	0    1    1    0
+$EndComp
+NoConn ~ 2000 2550
+NoConn ~ 3300 4350
+NoConn ~ 3300 3850
+NoConn ~ 3300 3550
+NoConn ~ 3300 3450
+$Comp
+L power:GND #PWR0106
+U 1 1 61ADEADE
+P 1800 3850
+F 0 "#PWR0106" H 1800 3600 50  0001 C CNN
+F 1 "GND" V 1900 3850 50  0000 C CNN
+F 2 "" H 1800 3850 50  0001 C CNN
+F 3 "" H 1800 3850 50  0001 C CNN
+	1    1800 3850
+	0    1    1    0
+$EndComp
+$Comp
+L HKUST_RT_RCL:R_Small_US R10
+U 1 1 61ADF9B2
+P 1900 3850
+F 0 "R10" V 1800 3850 50  0000 C CNN
+F 1 "10k" V 1800 3650 50  0000 C CNN
+F 2 "HKUST_RT_RCL:R_0805_2012Metric" H 1968 3759 50  0001 L CNN
+F 3 "" H 1900 3850 50  0001 C CNN
+	1    1900 3850
+	0    1    1    0
+$EndComp
