File: Hardware/ST-Link_v2-1/ST-Link_v2-1.sch (KiCad schematic (older format))
At the start: 39 parts, among them J1 Conn_01x06, P1 USB_C_Plug_USB2.0, U1 STM32F103CBTx, U2 LP5907MFX-3.3, Y1 8Mhz

Commit message: v2.2
Parts:
- removed D4: LED_Small, HKUST_RT_BJT:LED_0805_2012Metric, symbol HKUST_RT_BJT:LED_Small
- removed R10: 10k, HKUST_RT_RCL:R_0805_2012Metric, symbol HKUST_RT_RCL:R_Small_US
- removed R12: 1.5k, HKUST_RT_RCL:R_0805_2012Metric, symbol HKUST_RT_RCL:R_Small_US
- removed R8: 4.7k, HKUST_RT_RCL:R_0805_2012Metric, symbol HKUST_RT_RCL:R_Small_US
- R1: value 100k -> 10k
- R4, R5: value 1.5k -> 680R
Connections:
- wire segments 70 -> 66
- no-connect marks 19 -> 20
Other:
- moved on the sheet: D5
Changed lines of the file:
@@
 P 950 1300
 F 0 "R1" H 882 1254 50  0000 R CNN
-F 1 "100k" H 882 1345 50  0000 R CNN
+F 1 "10k" H 882 1345 50  0000 R CNN
 F 2 "HKUST_RT_RCL:R_0805_2012Metric" H 1018 1209 50  0001 L CNN
 F 3 "" H 950 1300 50  0001 C CNN
@@
 	0    -1   -1   0
 $EndComp
-$Comp
-L HKUST_RT_RCL:R_Small_US R8
-U 1 1 619766CF
-P 1800 3150
-F 0 "R8" V 1900 3150 50  0000 C CNN
-F 1 "4.7k" V 1900 3000 50  0000 C CNN
-F 2 "HKUST_RT_RCL:R_0805_2012Metric" H 1868 3059 50  0001 L CNN
-F 3 "" H 1800 3150 50  0001 C CNN
-	1    1800 3150
-	0    1    1    0
-$EndComp
-$Comp
-L HKUST_RT_RCL:R_Small_US R4
-U 1 1 6197CD50
-P 1750 6800
-F 0 "R4" V 1545 6800 50  0000 C CNN
-F 1 "1.5k" V 1636 6800 50  0000 C CNN
-F 2 "HKUST_RT_RCL:R_0805_2012Metric" H 1818 6709 50  0001 L CNN
-F 3 "" H 1750 6800 50  0001 C CNN
-	1    1750 6800
-	0    1    1    0
-$EndComp
-$Comp
-L HKUST_RT_BJT:LED_Small D2
-U 1 1 6197CD56
-P 1550 6800
-F 0 "D2" H 1800 6600 50  0000 C CNN
-F 1 "TX" H 1650 6700 50  0000 C CNN
-F 2 "HKUST_RT_BJT:LED_0805_2012Metric" V 1550 6800 50  0001 C CNN
-F 3 "" V 1550 6800 50  0001 C CNN
-	1    1550 6800
-	-1   0    0    1
-$EndComp
-$Comp
-L power:+3.3V #PWR07
-U 1 1 6197CD5C
-P 1450 6800
-F 0 "#PWR07" H 1450 6650 50  0001 C CNN
-F 1 "+3.3V" V 1465 6928 50  0000 L CNN
-F 2 "" H 1450 6800 50  0001 C CNN
-F 3 "" H 1450 6800 50  0001 C CNN
-	1    1450 6800
-	0    -1   -1   0
-$EndComp
-$Comp
-L HKUST_RT_RCL:R_Small_US R5
-U 1 1 6197E8BA
-P 1750 7150
-F 0 "R5" V 1545 7150 50  0000 C CNN
-F 1 "1.5k" V 1636 7150 50  0000 C CNN
-F 2 "HKUST_RT_RCL:R_0805_2012Metric" H 1818 7059 50  0001 L CNN
-F 3 "" H 1750 7150 50  0001 C CNN
-	1    1750 7150
-	0    1    1    0
-$EndComp
-$Comp
-L HKUST_RT_BJT:LED_Small D3
-U 1 1 6197E8C0
-P 1550 7150
-F 0 "D3" H 1800 6950 50  0000 C CNN
-F 1 "RX" H 1650 7050 50  0000 C CNN
-F 2 "HKUST_RT_BJT:LED_0805_2012Metric" V 1550 7150 50  0001 C CNN
-F 3 "" V 1550 7150 50  0001 C CNN
-	1    1550 7150
-	-1   0    0    1
-$EndComp
-$Comp
-L power:+3.3V #PWR08
-U 1 1 6197E8C6
-P 1450 7150
-F 0 "#PWR08" H 1450 7000 50  0001 C CNN
-F 1 "+3.3V" V 1465 7278 50  0000 L CNN
-F 2 "" H 1450 7150 50  0001 C CNN
-F 3 "" H 1450 7150 50  0001 C CNN
-	1    1450 7150
-	0    -1   -1   0
-$EndComp
-$Comp
-L HKUST_RT_BJT:LED_Small D5
-U 1 1 61984CA9
-P 3300 7050
-F 0 "D5" H 3300 6850 50  0000 C CNN
-F 1 "LED_Small" H 3450 6950 50  0000 C CNN
-F 2 "HKUST_RT_BJT:LED_0805_2012Metric" V 3300 7050 50  0001 C CNN
-F 3 "" V 3300 7050 50  0001 C CNN
-	1    3300 7050
-	1    0    0    -1
-$EndComp
-$Comp
-L HKUST_RT_RCL:R_Small_US R12
-U 1 1 61984F97
-P 3550 6800
-F 0 "R12" V 3345 6800 50  0000 C CNN
-F 1 "1.5k" V 3450 6800 50  0000 C CNN
-F 2 "HKUST_RT_RCL:R_0805_2012Metric" H 3618 6709 50  0001 L CNN
-F 3 "" H 3550 6800 50  0001 C CNN
-	1    3550 6800
-	0    1    1    0
-$EndComp
-$Comp
-L HKUST_RT_RCL:R_Small_US R11
-U 1 1 61985964
-P 3100 7050
-F 0 "R11" V 3000 7050 50  0000 C CNN
-F 1 "1.5k" V 3250 7000 50  0000 C CNN
-F 2 "HKUST_RT_RCL:R_0805_2012Metric" H 3168 6959 50  0001 L CNN
-F 3 "" H 3100 7050 50  0001 C CNN
-	1    3100 7050
-	0    1    1    0
-$EndComp
-$Comp
-L power:GND #PWR016
-U 1 1 61985E05
-P 3200 6800
-F 0 "#PWR016" H 3200 6550 50  0001 C CNN
-F 1 "GND" V 3100 6800 50  0000 R CNN
-F 2 "" H 3200 6800 50  0001 C CNN
-F 3 "" H 3200 6800 50  0001 C CNN
-	1    3200 6800
-	0    1    1    0
-$EndComp
-$Comp
-L power:+3.3V #PWR017
-U 1 1 61986DA2
-P 3400 7050
-F 0 "#PWR017" H 3400 6900 50  0001 C CNN
-F 1 "+3.3V" V 3415 7178 50  0000 L CNN
-F 2 "" H 3400 7050 50  0001 C CNN
-F 3 "" H 3400 7050 50  0001 C CNN
-	1    3400 7050
-	0    1    1    0
-$EndComp
 Wire Wire Line
 	5650 4750 5650 4850
@@
 $EndComp
 Wire Wire Line
-	3000 7050 3000 6650
-Wire Wire Line
-	3650 6650 3650 6800
-Connection ~ 3000 7050
-Wire Wire Line
 	1900 3050 2000 3050
-Wire Wire Line
-	1900 3150 2000 3150
 Wire Wire Line
 	1900 1950 2000 1950
@@
 	1    0    0    -1
 $EndComp
-Wire Wire Line
-	3400 6800 3450 6800
-Wire Wire Line
-	3000 6650 3650 6650
-Text Label 2550 7050 0    50   ~ 0
-LED_STLINK
-Wire Wire Line
-	2550 7050 3000 7050
-Wire Wire Line
-	2250 6800 1850 6800
-Wire Wire Line
-	2250 7150 1850 7150
-Text Label 2050 6800 0    50   ~ 0
-TXD
-Text Label 2050 7150 0    50   ~ 0
-RXD
 $Comp
 L HKUST_RT_RCL:R_Small_US R14
@@
 	0    1    1    0
 $EndComp
-Wire Wire Line
-	1700 2850 2000 2850
 Text Label 1350 1400 0    50   ~ 0
-NRST
-Text Label 1700 2850 0    50   ~ 0
 NRST
 Text Label 5900 6900 0    50   ~ 0
@@
 L power:+3.3V #PWR011
 U 1 1 619E13F6
-P 1700 3150
-F 0 "#PWR011" H 1700 3000 50  0001 C CNN
-F 1 "+3.3V" V 1700 3400 50  0000 C CNN
-F 2 "" H 1700 3150 50  0001 C CNN
-F 3 "" H 1700 3150 50  0001 C CNN
-	1    1700 3150
+P 1850 3150
+F 0 "#PWR011" H 1850 3000 50  0001 C CNN
+F 1 "+3.3V" V 1850 3400 50  0000 C CNN
+F 2 "" H 1850 3150 50  0001 C CNN
+F 3 "" H 1850 3150 50  0001 C CNN
+	1    1850 3150
 	0    -1   -1   0
 $EndComp
@@
 $EndComp
 $Comp
-L HKUST_RT_BJT:LED_Small D4
-U 1 1 61984398
-P 3300 6800
-F 0 "D4" H 3300 6900 50  0000 C CNN
-F 1 "LED_Small" H 3550 6700 50  0000 C CNN
-F 2 "HKUST_RT_BJT:LED_0805_2012Metric" V 3300 6800 50  0001 C CNN
-F 3 "" V 3300 6800 50  0001 C CNN
-	1    3300 6800
-	1    0    0    -1
-$EndComp
-$Comp
 L power:GND #PWR0104
 U 1 1 61AA0D72
@@
 NoConn ~ 3300 3450
 $Comp
-L power:GND #PWR0106
-U 1 1 61ADEADE
-P 1800 3850
-F 0 "#PWR0106" H 1800 3600 50  0001 C CNN
-F 1 "GND" V 1900 3850 50  0000 C CNN
-F 2 "" H 1800 3850 50  0001 C CNN
-F 3 "" H 1800 3850 50  0001 C CNN
-	1    1800 3850
-	0    1    1    0
-$EndComp
-$Comp
-L HKUST_RT_RCL:R_Small_US R10
-U 1 1 61ADF9B2
-P 1900 3850
-F 0 "R10" V 1800 3850 50  0000 C CNN
-F 1 "10k" V 1800 3650 50  0000 C CNN
-F 2 "HKUST_RT_RCL:R_0805_2012Metric" H 1968 3759 50  0001 L CNN
-F 3 "" H 1900 3850 50  0001 C CNN
-	1    1900 3850
-	0    1    1    0
-$EndComp
-$Comp
 L power:+5V #PWR0103
 U 1 1 619F8999
@@
 	5350 2750 5650 2750
 Connection ~ 5650 2750
+Wire Wire Line
+	2550 7050 3000 7050
+Text Label 2550 7050 0    50   ~ 0
+LED_STLINK
+$Comp
+L HKUST_RT_RCL:R_Small_US R11
+U 1 1 61985964
+P 3100 7050
+F 0 "R11" V 3000 7050 50  0000 C CNN
+F 1 "1.5k" V 3250 7000 50  0000 C CNN
+F 2 "HKUST_RT_RCL:R_0805_2012Metric" H 3168 6959 50  0001 L CNN
+F 3 "" H 3100 7050 50  0001 C CNN
+	1    3100 7050
+	0    1    1    0
+$EndComp
+$Comp
+L HKUST_RT_BJT:LED_Small D5
+U 1 1 61984CA9
+P 3300 7050
+F 0 "D5" H 3300 6850 50  0000 C CNN
+F 1 "LED_Small" H 3150 6950 50  0000 C CNN
+F 2 "HKUST_RT_BJT:LED_0805_2012Metric" V 3300 7050 50  0001 C CNN
+F 3 "" V 3300 7050 50  0001 C CNN
+	1    3300 7050
+	-1   0    0    1
+$EndComp
+Text Label 2050 7150 0    50   ~ 0
+RXD
+Text Label 2050 6800 0    50   ~ 0
+TXD
+Wire Wire Line
+	2250 7150 1850 7150
+Wire Wire Line
+	2250 6800 1850 6800
+$Comp
+L power:+3.3V #PWR08
+U 1 1 6197E8C6
+P 1450 7150
+F 0 "#PWR08" H 1450 7000 50  0001 C CNN
+F 1 "+3.3V" V 1465 7278 50  0000 L CNN
+F 2 "" H 1450 7150 50  0001 C CNN
+F 3 "" H 1450 7150 50  0001 C CNN
+	1    1450 7150
+	0    -1   -1   0
+$EndComp
+$Comp
+L HKUST_RT_BJT:LED_Small D3
+U 1 1 6197E8C0
+P 1550 7150
+F 0 "D3" H 1800 6950 50  0000 C CNN
+F 1 "RX" H 1650 7050 50  0000 C CNN
+F 2 "HKUST_RT_BJT:LED_0805_2012Metric" V 1550 7150 50  0001 C CNN
+F 3 "" V 1550 7150 50  0001 C CNN
+	1    1550 7150
+	-1   0    0    1
+$EndComp
+$Comp
+L HKUST_RT_RCL:R_Small_US R5
+U 1 1 6197E8BA
+P 1750 7150
+F 0 "R5" V 1545 7150 50  0000 C CNN
+F 1 "680R" V 1636 7150 50  0000 C CNN
+F 2 "HKUST_RT_RCL:R_0805_2012Metric" H 1818 7059 50  0001 L CNN
+F 3 "" H 1750 7150 50  0001 C CNN
+	1    1750 7150
+	0    1    1    0
+$EndComp
+$Comp
+L power:+3.3V #PWR07
+U 1 1 6197CD5C
+P 1450 6800
+F 0 "#PWR07" H 1450 6650 50  0001 C CNN
+F 1 "+3.3V" V 1465 6928 50  0000 L CNN
+F 2 "" H 1450 6800 50  0001 C CNN
+F 3 "" H 1450 6800 50  0001 C CNN
+	1    1450 6800
+	0    -1   -1   0
+$EndComp
+$Comp
+L HKUST_RT_BJT:LED_Small D2
+U 1 1 6197CD56
+P 1550 6800
+F 0 "D2" H 1800 6600 50  0000 C CNN
+F 1 "TX" H 1650 6700 50  0000 C CNN
+F 2 "HKUST_RT_BJT:LED_0805_2012Metric" V 1550 6800 50  0001 C CNN
+F 3 "" V 1550 6800 50  0001 C CNN
+	1    1550 6800
+	-1   0    0    1
+$EndComp
+$Comp
+L HKUST_RT_RCL:R_Small_US R4
+U 1 1 6197CD50
+P 1750 6800
+F 0 "R4" V 1545 6800 50  0000 C CNN
+F 1 "680R" V 1636 6800 50  0000 C CNN
+F 2 "HKUST_RT_RCL:R_0805_2012Metric" H 1818 6709 50  0001 L CNN
+F 3 "" H 1750 6800 50  0001 C CNN
+	1    1750 6800
+	0    1    1    0
+$EndComp
+$Comp
+L power:GND #PWR0105
+U 1 1 61C99FE1
+P 3400 7050
+F 0 "#PWR0105" H 3400 6800 50  0001 C CNN
+F 1 "GND" V 3405 6922 50  0000 R CNN
+F 2 "" H 3400 7050 50  0001 C CNN
+F 3 "" H 3400 7050 50  0001 C CNN
+	1    3400 7050
+	0    -1   -1   0
+$EndComp
+NoConn ~ 2000 2850
+Wire Wire Line
+	2000 3850 1850 3850
+Wire Wire Line
+	2000 3150 1850 3150
+$Comp
+L power:GND #PWR0106
+U 1 1 61ADEADE
+P 1850 3850
+F 0 "#PWR0106" H 1850 3600 50  0001 C CNN
+F 1 "GND" V 1950 3700 50  0000 C CNN
+F 2 "" H 1850 3850 50  0001 C CNN
+F 3 "" H 1850 3850 50  0001 C CNN
+	1    1850 3850
+	0    1    1    0
+$EndComp
 $EndSCHEMATC
