File: Hardware/ST-Link_v2-1/ST-Link_v2-1.kicad_pcb (KiCad board)
At the start: 2 copper layers, 40 parts, among them J1 Conn_01x06, J2 USB_C_Male, U1 STM32F103CBTx, U2 LP5907MFX-3.3, Y1 8MHz

Commit message: 1.1
Parts:
- C1, C2, C3, C4, C5, C6, C7, R1, R13, R15, R16, R19, R2, R20, R3, R4, R5, R6, R7, R8, U2, Y1: moved to B.Cu
- moved D5 34.4 mm to (173.6, 106.9), turned to 45 degrees
- moved D3 34.4 mm to (183.9, 105.8), turned to 180 degrees
- moved D4 34.4 mm to (172.8, 106.2), turned to 225 degrees
- moved C1 32.5 mm to (179.3, 107.8), turned to 270 degrees
- moved C5 31.9 mm to (176.8, 105.8)
- moved C3 30.6 mm to (181.2, 109.2), turned to 180 degrees
- moved R11 29.1 mm to (173.0, 109.7), turned to 270 degrees
- moved R16 28.8 mm to (172.5, 112.3)
- moved R17 28.8 mm to (172.5, 111.3)
- moved R12 28.7 mm to (172.0, 109.7), turned to 90 degrees
- moved C8 27.7 mm to (172.4, 113.8)
- moved C6 26.9 mm to (176.1, 113.0), turned to 90 degrees
- moved C9 26.9 mm to (174.0, 115.6), turned to 180 degrees
- moved R7 25.4 mm to (178.3, 107.8), turned to 90 degrees
- moved C2 24.7 mm to (181.2, 114.6), turned to 180 degrees
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Routing:
- net +3V3: track 0.00 -> 56.0 mm, vias 0 -> 6
- net /SWCLK: track 0.00 -> 29.1 mm, vias 0 -> 5
- net +5V: track 0.00 -> 26.9 mm, vias 0 -> 3
- net /SWDIO: track 0.00 -> 18.5 mm, vias 0 -> 2
- net /TXD: track 0.00 -> 13.1 mm, vias 0 -> 2
- net /RXD: track 0.00 -> 9.64 mm, vias 0 -> 2
- net /NRST: track 0.00 -> 8.68 mm, vias 0 -> 2
- net Net-(D6-Pad1): track 0.00 -> 6.37 mm
- net Net-(C2-Pad1): track 0.00 -> 4.04 mm, vias 0 -> 1
- net Net-(C3-Pad1): track 0.00 -> 4.01 mm, vias 0 -> 1
- net /LED_STLINK: track 0.00 -> 3.27 mm
- net Net-(D4-Pad2): track 0.00 -> 2.93 mm
- net /ST_SWDIO: track 0.00 -> 2.48 mm, vias 0 -> 1
- net /ST_SWCLK: track 0.00 -> 2.28 mm, vias 0 -> 1
- net Net-(R10-Pad1): track 0.00 -> 2.28 mm
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- added copper zone on B.Cu, net GND
- added copper zone on F.Cu, net GND
Other:
- board outline added: 22.7 x 14 mm
- net class Default: trace_width 0.25 -> 0.254; via_dia 0.8 -> 0.508; via_drill 0.4 -> 0.3048
- rule via_min_drill: 0.3 -> 0.3048
- rule via_min_size: 0.4 -> 0.4064

Commit message: 1.2
Parts:
- C9: moved to B.Cu
- U2: moved to F.Cu
- moved R3 3.94 mm to (170.1, 117.1), turned to 0 degrees
- moved D1 3.49 mm to (170.6, 117.6), turned to 270 degrees
- moved R2 2.41 mm to (173.7, 109.0)
- moved U2 2.05 mm to (173.1, 116.7), turned to 270 degrees
- moved C6 1.10 mm to (175.5, 113.9), turned to 180 degrees
- moved C9 1.03 mm to (174.1, 116.6), turned to 90 degrees
- moved R20 0.89 mm to (176.1, 111.9), turned to 270 degrees
- moved R19 0.42 mm to (177.4, 113.4)
Routing:
- net +3V3: track 56.0 -> 70.8 mm, vias 6 -> 8
- net /SWCLK: track 29.1 -> 22.8 mm, vias 5 -> 4
- net +5V: track 26.9 -> 25.1 mm, vias 3 -> 2
- net /SWDIO: track 18.5 -> 20.2 mm
- net GND: vias 8 -> 11

Commit message: 1.2.2
Routing:
- net GND: vias 11 -> 19
Other:
- board text added: "24/11/2021 V1.2"
- board text added: "HKUST Robotics Team"
- board text added: "ST-LinkV2-1"
- board text added: "by Samson"

Commit message: v2 2/12/2021
Parts:
- added R21: 5.1k, HKUST_RT_RCL:R_0805_2012Metric_Pad1.20x1.40mm_HandSolder, F.Cu at (182.6, 140.3)
- C1, C2, C3, C4, C5, C6, C7, C9: footprint HKUST_RT_RCL:C_0402_1005Metric -> HKUST_RT_RCL:C_0805_2012Metric_Pad1.18x1.45mm_HandSolder
- C8: footprint HKUST_RT_RCL:C_0402_1005Metric -> HKUST_RT_RCL:C_0805_2012Metric_Pad1.18x1.45mm_HandSolder; moved to B.Cu
- D1, D2, D3, D4, D5: footprint HKUST_RT_BJT:LED_0402_1005Metric -> HKUST_RT_BJT:LED_0805_2012Metric_Pad1.15x1.40mm_HandSolder
- D6: footprint HKUST_RT_BJT:D_0402_1005Metric -> HKUST_RT_BJT:D_SOD-123
- R1, R4, R5: footprint HKUST_RT_RCL:R_0402_1005Metric -> HKUST_RT_RCL:R_0805_2012Metric_Pad1.20x1.40mm_HandSolder; moved to F.Cu
- R10, R14, R9: footprint HKUST_RT_RCL:R_0402_1005Metric -> HKUST_RT_RCL:R_0805_2012Metric_Pad1.20x1.40mm_HandSolder; moved to B.Cu
- R11, R12, R13, R15, R16, R17, R18, R2, R3, R6, R7, R8: footprint HKUST_RT_RCL:R_0402_1005Metric -> HKUST_RT_RCL:R_0805_2012Metric_Pad1.20x1.40mm_HandSolder
- Y1: moved to F.Cu
- moved C5 40.8 mm to (192.4, 143.5), turned to 180 degrees
- moved R3 39.6 mm to (198.0, 145.2)
- moved D1 38.9 mm to (198.0, 145.2), turned to 180 degrees
- moved R1 35.3 mm to (197.9, 135.5), turned to 0 degrees
- moved C4 34.4 mm to (197.9, 142.1)
- moved C1 33.3 mm to (197.9, 135.5), turned to 0 degrees
- moved C8 33.0 mm to (182.6, 145.2), turned to 180 degrees
- moved C3 33.0 mm to (197.9, 137.7), turned to 0 degrees
- moved Y1 31.9 mm to (197.9, 138.8)
- moved D4 31.8 mm to (202.1, 118.7), turned to 0 degrees
- moved J1 31.5 mm to (203.5, 139.2)
- moved R6 31.4 mm to (192.4, 145.5), turned to 0 degrees
- moved R13 30.7 mm to (188.5, 144.6), turned to 270 degrees
- moved C2 30.4 mm to (197.9, 140.0), turned to 0 degrees
- moved U2 29.8 mm to (184.8, 144.1), turned to 90 degrees
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Connections:
- D6 pad 1: Net-(D6-Pad1) -> +5V
- D6 pad 2: +5V -> Net-(D6-Pad2)
- J1 pad 1: Net-(D6-Pad1) -> +5V
- J2 pad A4: +5V -> Net-(D6-Pad2)
- J2 pad A9: +5V -> Net-(D6-Pad2)
- J2 pad B4: +5V -> Net-(D6-Pad2)
- J2 pad B9: +5V -> Net-(D6-Pad2)
Routing:
- net +3V3: track 70.8 -> 0.00 mm, vias 8 -> 0
- net +5V: track 25.1 -> 0.00 mm, vias 2 -> 0
- net /SWCLK: track 22.8 -> 0.00 mm, vias 4 -> 0
- net /SWDIO: track 20.2 -> 0.00 mm, vias 2 -> 0
- net /TXD: track 13.6 -> 0.00 mm, vias 2 -> 0
- net /RXD: track 9.56 -> 0.00 mm, vias 2 -> 0
- net /NRST: track 9.13 -> 0.00 mm, vias 2 -> 0
- net Net-(D6-Pad1): track 6.37 -> 0.00 mm
- net Net-(C2-Pad1): track 4.04 -> 0.00 mm, vias 1 -> 0
- net Net-(C3-Pad1): track 4.01 -> 0.00 mm, vias 1 -> 0
- net /LED_STLINK: track 3.27 -> 0.00 mm
- net Net-(D4-Pad2): track 2.93 -> 0.00 mm
- net /ST_SWDIO: track 2.56 -> 0.00 mm, vias 1 -> 0
- net /ST_SWCLK: track 2.30 -> 0.00 mm, vias 1 -> 0
- net Net-(R10-Pad1): track 2.28 -> 0.00 mm
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- removed copper zone on B.Cu, net GND
- removed copper zone on F.Cu, net GND
Other:
- board size 22.7 x 14 mm -> 30.4 x 15 mm
- board text removed: "24/11/2021 V1.2"
- board text removed: "HKUST Robotics Team"
- board text removed: "ST-LinkV2-1"
- board text removed: "by Samson"

Commit message: find bug in sch
Parts:
- added R22: 5.1k, HKUST_RT_RCL:R_0805_2012Metric, B.Cu at (182.0, 136.3)
- C1, C2, C3, C4, C5, C6, C7, C8, C9: footprint HKUST_RT_RCL:C_0805_2012Metric_Pad1.18x1.45mm_HandSolder -> HKUST_RT_RCL:C_0805_2012Metric
- D1, D2, D3, D4, D5: footprint HKUST_RT_BJT:LED_0805_2012Metric_Pad1.15x1.40mm_HandSolder -> HKUST_RT_BJT:LED_0805_2012Metric
- J2: value USB_C_Male -> USB_C_Receptacle
- R1, R11, R12, R21: footprint HKUST_RT_RCL:R_0805_2012Metric_Pad1.20x1.40mm_HandSolder -> HKUST_RT_RCL:R_0805_2012Metric; moved to B.Cu
- R10, R14, R15, R16, R17, R18, R3, R4, R5, R8: footprint HKUST_RT_RCL:R_0805_2012Metric_Pad1.20x1.40mm_HandSolder -> HKUST_RT_RCL:R_0805_2012Metric
- R13, R2, R6, R9: footprint HKUST_RT_RCL:R_0805_2012Metric_Pad1.20x1.40mm_HandSolder -> HKUST_RT_RCL:R_0805_2012Metric; moved to F.Cu
- R19, R20: footprint HKUST_RT_RCL:R_0402_1005Metric -> HKUST_RT_RCL:R_0805_2012Metric
- R7: value 100R -> 10k; footprint HKUST_RT_RCL:R_0805_2012Metric_Pad1.20x1.40mm_HandSolder -> HKUST_RT_RCL:R_0805_2012Metric
- Y1: value 8MHz -> 8Mhz
- moved R5 32.1 mm to (192.7, 129.8)
- moved D3 31.4 mm to (196.1, 129.8)
- moved D2 29.7 mm to (196.1, 131.8), turned to 180 degrees
- moved R12 23.0 mm to (183.3, 133.5), turned to 90 degrees
- moved D4 22.3 mm to (183.5, 131.1), turned to 225 degrees
- moved R4 20.2 mm to (196.1, 133.9)
- moved D1 18.7 mm to (179.3, 143.6), turned to 270 degrees
- moved R3 18.7 mm to (179.3, 143.6), turned to 90 degrees
- moved R11 16.0 mm to (181.2, 133.5), turned to 270 degrees
- moved C5 15.5 mm to (184.9, 129.9)
- moved C7 11.5 mm to (191.1, 142.3)
- moved D5 11.3 mm to (180.9, 130.7), turned to 45 degrees
- moved R1 11.0 mm to (188.3, 129.9), turned to 180 degrees
- moved C4 10.6 mm to (191.1, 134.0), turned to 90 degrees
- moved C1 8.27 mm to (191.8, 129.9)
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Connections:
- J1 pad 2: /SWDIO -> /SWCLK
- J1 pad 3: /SWCLK -> /SWDIO
- J2 pad B6: (no net) -> Net-(J2-PadA6)
- J2 pad B7: (no net) -> Net-(J2-PadA7)
- J2 pad S2: GND -> (no net)
- J2 pad S3: GND -> (no net)
- J2 pad S4: GND -> (no net)
- R13 pad 2: GND -> +3V3
- R16 pad 1: Net-(J2-PadA6) -> +3V3
- R16 pad 2: +3V3 -> /D+
- R17 pad 1: Net-(J2-PadA7) -> /D-
- R17 pad 2: /D- -> Net-(J2-PadA7)
- R18 pad 1: Net-(J2-PadA6) -> /D+
- R18 pad 2: /D+ -> Net-(J2-PadA6)
- Y1 pad 1: Net-(C3-Pad1) -> Net-(C2-Pad1)
- Y1 pad 2: Net-(C2-Pad1) -> GND
- Y1 pad 3: (no net) -> Net-(C3-Pad1)
- Y1 pad 4: (no net) -> GND
Routing:
- net /SWDIO: track 0.00 -> 4.76 mm, vias 0 -> 1
- net /SWDIO_IN: track 0.00 -> 4.74 mm
- net Net-(D6-Pad2): track 0.00 -> 3.78 mm
- net Net-(R9-Pad1): track 0.00 -> 3.63 mm
- net +5V: track 0.00 -> 3.33 mm, vias 0 -> 1
- net +3V3: track 0.00 -> 3.23 mm, vias 0 -> 1
- net Net-(J2-PadA7): track 0.00 -> 2.58 mm
- net Net-(J2-PadA6): track 0.00 -> 2.40 mm
- net /D+: track 0.00 -> 2.23 mm
- net Net-(J2-PadB5): track 0.00 -> 2.19 mm
- net /D-: track 0.00 -> 2.17 mm
- net /ST_SWDIO: track 0.00 -> 1.38 mm, vias 0 -> 1
- net Net-(D4-Pad2): track 0.00 -> 0.63 mm
- net Net-(D1-Pad1): vias 0 -> 1
- added copper zone on B.Cu, net GND
- added copper zone on F.Cu, net GND
Other:
- board size 30.4 x 15 mm -> 26.3 x 17.7 mm

Commit message: 5/12/2021
Parts:
- removed D6: 1N4001, HKUST_RT_BJT:D_SOD-123
- removed R13: 100R, HKUST_RT_RCL:R_0805_2012Metric
- C8, R10, R8: moved to F.Cu
- R14, R15: value 4.7k -> 10k
- moved R10 13.8 mm to (189.1, 129.8), turned to 0 degrees
- moved C8 2.84 mm to (184.0, 140.5), turned to 0 degrees
- moved C7 2.65 mm to (191.3, 139.7)
- moved C9 1.92 mm to (184.0, 144.4), turned to 180 degrees
- moved R9 1.74 mm to (195.8, 141.1)
- moved D1 1.66 mm to (181.0, 143.8)
- moved R3 1.65 mm to (181.0, 143.7)
- moved R6 1.31 mm to (192.2, 143.0)
- moved R8 1.31 mm to (188.7, 143.0)
- moved R7 1.17 mm to (189.1, 132.6), turned to 90 degrees
- moved C1 1.02 mm to (192.8, 129.8)
- moved R19 0.89 mm to (189.1, 136.9)
- moved R20 0.89 mm to (187.1, 136.9)
- moved U2 0.83 mm to (184.0, 143.5), turned to 270 degrees
- moved C6 0.83 mm to (187.8, 139.7)
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Connections:
- net /SWCLK renamed /JTCK
- net /SWDIO renamed /JTMS
- net /SWDIO_IN renamed Net-(R2-Pad1)
- J2 pad A4: Net-(D6-Pad2) -> +5V
- J2 pad A9: Net-(D6-Pad2) -> +5V
- J2 pad B4: Net-(D6-Pad2) -> +5V
- J2 pad B9: Net-(D6-Pad2) -> +5V
- U1 pad 21: Net-(U1-Pad21) -> Net-(R10-Pad1)
- U1 pad 3: Net-(R10-Pad1) -> Net-(U1-Pad3)
Routing:
- net +3V3: track 3.23 -> 31.8 mm, vias 1 -> 3
- net +5V: track 3.33 -> 27.6 mm, vias 1 -> 3
- net /LED_STLINK: track 0.00 -> 8.75 mm, vias 0 -> 1
- net /JTCK: track 0.00 -> 4.98 mm, vias 0 -> 1
- net Net-(J2-PadA5): track 0.00 -> 4.80 mm, vias 0 -> 1
- net Net-(J2-PadA7): track 2.58 -> 7.09 mm, vias 0 -> 2
- net /ST_SWCLK: track 0.00 -> 4.11 mm, vias 0 -> 1
- net Net-(D6-Pad2): track 3.78 -> 0.00 mm
- net Net-(R9-Pad1): track 3.63 -> 0.00 mm
- net Net-(R6-Pad1): track 0.00 -> 3.06 mm
- net Net-(R8-Pad1): track 0.00 -> 2.78 mm
- net Net-(R7-Pad1): track 0.00 -> 1.60 mm, vias 0 -> 1
- net Net-(J2-PadB5): track 2.19 -> 3.07 mm
- net Net-(J2-PadA6): track 2.40 -> 3.14 mm
- net Net-(D5-Pad1): track 0.48 -> 1.13 mm, vias 0 -> 1
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Other:
- board size 26.3 x 17.7 mm -> 27.6 x 17.7 mm

Commit message: V2.1 11/12/2021
Parts:
- removed J2: USB_C_Receptacle, HKUST_RT_CONN:USB_C_MALE
- removed R21: 5.1k, HKUST_RT_RCL:R_0805_2012Metric
- added P1: USB_C_Plug_USB2.0, HKUST_RT_CONN:USB_C_MALE, F.Cu at (122.7, 90.0)
- C8, R10, R2, R4, R5, R6, R8, R9, Y1: moved to B.Cu
- moved C6 77.4 mm to (132.4, 85.6)
- moved C4 76.4 mm to (128.8, 90.7)
- moved C9 75.9 mm to (126.0, 95.4)
- moved U2 75.9 mm to (126.0, 94.6)
- moved J1 75.4 mm to (143.0, 89.5)
- moved R8 74.6 mm to (131.7, 94.9), turned to 90 degrees
- moved C8 74.6 mm to (126.0, 93.5)
- moved R14 74.3 mm to (141.9, 83.7)
- moved R12 74.0 mm to (126.0, 86.9), turned to 180 degrees
- moved R17 74.0 mm to (126.0, 88.8)
- moved R22 74.0 mm to (126.0, 88.8)
- moved C7 74.0 mm to (137.2, 89.3), turned to 270 degrees
- moved R11 73.7 mm to (126.0, 85.0), turned to 0 degrees
- moved R16 73.7 mm to (126.0, 91.3)
- moved R18 73.7 mm to (126.0, 91.3)
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Routing:
- net +5V: track 27.6 -> 86.4 mm
- net +3V3: track 31.8 -> 82.1 mm, vias 3 -> 10
- net /RXD: track 0.00 -> 35.9 mm, vias 0 -> 1
- net /JTMS: track 4.89 -> 34.8 mm, vias 1 -> 2
- net /TXD: track 0.00 -> 27.0 mm, vias 0 -> 1
- net Net-(R6-Pad1): track 3.06 -> 23.2 mm, vias 0 -> 1
- net /NRST: track 0.00 -> 12.6 mm, vias 0 -> 1
- net /JTCK: track 4.98 -> 17.4 mm, vias 1 -> 3
- net Net-(C3-Pad1): track 0.00 -> 9.03 mm, vias 0 -> 1
- net Net-(R14-Pad1): track 0.00 -> 8.31 mm, vias 0 -> 1
- net Net-(R7-Pad1): track 1.60 -> 7.30 mm
- net Net-(J2-PadA5): track 4.80 -> 0.00 mm, vias 1 -> 0
- net Net-(R9-Pad1): track 0.00 -> 4.75 mm, vias 0 -> 1
- net Net-(C2-Pad1): track 0.00 -> 4.37 mm, vias 0 -> 1
- net Net-(P1-PadA7): track 7.09 -> 3.27 mm, vias 2 -> 0
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Other:
- board size 27.6 x 17.7 mm -> 26.3 x 19 mm
- board text added: "11/12/2021"
- board text added: "3.3V"
- board text added: "HKUST Robotics Team"
- board text added: "RX"
- board text added: "ST-Link-V2 V2.1"
- board text added: "TX"
- board text added: "by Samson"

Commit message: v2.2
Parts:
- removed D4: LED_Small, HKUST_RT_BJT:LED_0805_2012Metric
- removed R10: 10k, HKUST_RT_RCL:R_0805_2012Metric
- removed R12: 1.5k, HKUST_RT_RCL:R_0805_2012Metric
- removed R8: 4.7k, HKUST_RT_RCL:R_0805_2012Metric
- R1: value 100k -> 10k
- R4, R5: value 1.5k -> 680R
- moved D5 0.76 mm to (126.0, 85.7), turned to 90 degrees
- moved R11 0.76 mm to (126.0, 85.7), turned to 270 degrees
Connections:
- D5 pad 1: Net-(D5-Pad1) -> GND
- D5 pad 2: +3V3 -> Net-(D5-Pad2)
- R11 pad 1: Net-(D5-Pad1) -> Net-(D5-Pad2)
- U1 pad 18: /NRST -> Net-(U1-Pad18)
- U1 pad 21: Net-(R10-Pad1) -> GND
- U1 pad 39: Net-(R8-Pad1) -> +3V3
Routing:
- net Net-(R6-Pad1): track 23.2 -> 15.5 mm
- net +3V3: track 82.1 -> 78.3 mm
- net Net-(R8-Pad1): track 2.90 -> 0.00 mm, vias 1 -> 0
- net Net-(R10-Pad1): track 2.63 -> 0.00 mm, vias 1 -> 0
- net GND: track 0.00 -> 2.63 mm, vias 16 -> 17
- net /LED_STLINK: track 7.55 -> 4.98 mm
- net /NRST: track 12.6 -> 10.4 mm, vias 1 -> 2
- net Net-(D5-Pad2): vias 0 -> 1
- net Net-(D5-Pad1): vias 1 -> 0
- net Net-(D4-Pad2): vias 1 -> 0
Other:
- board text added: "26/12/2021"
- board text added: "ST-Link-V2 V2.2"
- board text removed: "11/12/2021"
- board text removed: "ST-Link-V2 V2.1"
